Commit message: changed urdf for pr2 to include transmissions

File: pr2_billiards_sim/urdf/pr2.urdf.xacro (robot description, xacro)
@@ -163,4 +163,5 @@
     <axis xyz="0 1 0"/>
     <limit lower="0" upper="1.8" effort="10000" velocity="1.0"/>
+    <calibration reference_position="0.0"/>
   </joint>
   <link name="cue_stick">
@@ -197,4 +198,5 @@
     <axis xyz="0 0 1"/>
     <limit lower="-0.1" upper="0.1" effort="10000" velocity="1.0"/>
+    <calibration reference_position="0.0"/>
   </joint>
   <link name="bridge">
@@ -251,3 +253,13 @@
     <selfCollide>true</selfCollide>
   </gazebo>
+<transmission name="lever_cue" type="SimpleTransmission">
+<actuator name="lc"/>
+<joint name="cue_ball_joint"/>
+<mechanicalReduction>1.0</mechanicalReduction>
+</transmission>
+<transmission name="cue_bridge" type="SimpleTransmission">
+<actuator name="cb"/>
+<joint name="cue_bridge_joint"/>
+<mechanicalReduction>1.0</mechanicalReduction>
+</transmission>
 </robot>

Commit message: urdf changed, left arm ik added,  ReadME created

File: pr2_billiards_sim/urdf/pr2.urdf.xacro (robot description, xacro)
@@ -150,17 +150,17 @@
     <turnGravityOff>false</turnGravityOff>
   </gazebo>
-  <xacro:property name="cue_length" value="0.8"/>
-  <xacro:property name="cue_radius" value="0.0075"/>
-  <xacro:property name="cue_mass" value="0.1"/>
-  <xacro:property name="cue_ixx" value="0.1"/>
-  <xacro:property name="cue_iyy" value="0.1"/>
-  <xacro:property name="cue_izz" value="0.01"/>
+  <xacro:property name="cue_length" value="1.47"/>
+  <xacro:property name="cue_radius" value="0.0065"/>
+  <xacro:property name="cue_mass" value="0.01"/>
+  <xacro:property name="cue_ixx" value="0.01"/>
+  <xacro:property name="cue_iyy" value="0.01"/>
+  <xacro:property name="cue_izz" value="0.001"/>
   <xacro:property name="cue_offset_z" value="0.03"/>
   <joint name="cue_ball_joint" type="revolute" >
     <parent link="lever_stick" />
     <child link="cue_stick" />
-    <origin xyz="0 0 ${lever_length}" rpy="0 0 0" />
+    <origin xyz="-0.4 0 ${lever_length}" rpy="0 0 0" />
     <axis xyz="0 1 0"/>
-    <limit lower="0" upper="1.8" effort="10000" velocity="1.0"/>
+    <limit lower="0.0" upper="1.8" effort="10000" velocity="1.0"/>
     <calibration reference_position="0.0"/>
   </joint>
@@ -195,6 +195,6 @@
     <parent link="cue_stick" />
     <child link="bridge" />
-    <origin xyz="0 0 ${cue_length-0.05}" rpy="0 0 0" />
-    <axis xyz="0 0 1"/>
+    <origin xyz="0 0 ${cue_length-0.05}" rpy="1.57 0 0" />
+    <axis xyz="0 1 0"/>
     <limit lower="-0.1" upper="0.1" effort="10000" velocity="1.0"/>
     <calibration reference_position="0.0"/>
@@ -209,5 +209,5 @@
       <origin xyz="-0.06 0 0" rpy="0 0 0" />
       <geometry>
-        <box size="0.10 0.03 0.005"/>
+        <box size="0.10 0.04 0.005"/>
       </geometry>
     </visual>

File: pr2_billiards_sim/urdf/table.urdf.xacro (robot description, xacro)
@@ -5,13 +5,13 @@
        xmlns:controller="http://playerstage.sourceforge.net/gazebo/xmlschema/#controller"
        xmlns:interface="http://playerstage.sourceforge.net/gazebo/xmlschema/#interface">
-  <xacro:property name="table_width" value="1.2192"/> <!-- 4ft -->
-  <xacro:property name="table_length" value="2.4384"/> <!-- 8ft -->
+  <xacro:property name="table_width" value="1.3592"/> <!-- 4ft -->
+  <xacro:property name="table_length" value="2.4784"/> <!-- 8ft -->
   <xacro:property name="table_height" value=".05"/>
-  <xacro:property name="side_pocket_dl" value="0.18"/>
-  <xacro:property name="corner_pocket_dw" value="0.08"/>
-  <xacro:property name="corner_pocket_dl" value="0.08"/>
-  <xacro:property name="cushion_height" value="0.05"/>
-  <xacro:property name="cushion_size" value="0.05"/>
-  <xacro:property name="leg_height" value="0.7"/>
+  <xacro:property name="side_pocket_dl" value="0.14"/>
+  <xacro:property name="corner_pocket_dw" value="0.12"/>
+  <xacro:property name="corner_pocket_dl" value="0.12"/>
+  <xacro:property name="cushion_height" value="0.035"/>
+  <xacro:property name="cushion_size" value="0.12"/>
+  <xacro:property name="leg_height" value="0.72"/>
   <!-- x along the long side, y short side, z up and origin at surface of table top -->
   <link name="pool_table">
@@ -36,6 +36,6 @@
   <gazebo reference="pool_table">
     <material>Gazebo/Green</material>
-    <mu1>1.0</mu1>
-    <mu2>1.0</mu2>
+    <mu1>100.0</mu1>
+    <mu2>100.0</mu2>
   </gazebo>
    <!-- with origin at final approach -->

Commit message: readme added

File: pr2_billiards_sim/urdf/pr2.urdf.xacro (robot description, xacro)
@@ -149,4 +149,5 @@
     <material>Gazebo/Wood</material>
     <turnGravityOff>false</turnGravityOff>
+    <selfCollide>true</selfCollide>
   </gazebo>
   <xacro:property name="cue_length" value="1.47"/>
@@ -187,4 +188,5 @@
     <material>Gazebo/Wood</material>
     <turnGravityOff>false</turnGravityOff>
+    <selfCollide>true</selfCollide>
   </gazebo>
   <xacro:property name="bridge_mass" value="0.1"/>
@@ -209,5 +211,5 @@
       <origin xyz="-0.06 0 0" rpy="0 0 0" />
       <geometry>
-        <box size="0.10 0.04 0.005"/>
+        <box size="0.10 0.04 0.01"/>
       </geometry>
     </visual>
@@ -215,5 +217,5 @@
       <origin xyz="-0.06 0 0" rpy="0 0 0" />
       <geometry>
-        <box size="0.10 0.03 0.005"/>
+        <box size="0.10 0.04 0.01"/>
       </geometry>
     </collision>
@@ -221,5 +223,7 @@
   <gazebo reference="bridge">
     <material>Gazebo/White</material>
-    <turnGravityOff>false</turnGravityOff>
+    <turnGravityOff>true</turnGravityOff>
+    <mu1>100.0</mu1>
+    <mu2>100.0</mu2>
     <selfCollide>true</selfCollide>
   </gazebo>
@@ -258,8 +262,8 @@
 <mechanicalReduction>1.0</mechanicalReduction>
 </transmission>
-<transmission name="cue_bridge" type="SimpleTransmission">
+<!--transmission name="cue_bridge" type="SimpleTransmission">
 <actuator name="cb"/>
 <joint name="cue_bridge_joint"/>
 <mechanicalReduction>1.0</mechanicalReduction>
-</transmission>
+</transmission-->
 </robot>

Commit message: Separated stick fvrom robot

File: pr2_billiards_sim/urdf/pr2.urdf.xacro (robot description, xacro)
@@ -13,5 +13,5 @@
   <include filename="$(find pr2_description)/urdf/forearm_v0/forearm.urdf.xacro" />
   <!-- PR2 gripper -->
-  <include filename="$(find pr2_description)/urdf/gripper_v0/gripper.urdf.xacro" />
+  <include filename="$(find pr2_billiards_sim)/urdf/ashok/gripper_v0/gripper.urdf.xacro" />
   <!-- PR2 head -->
   <include filename="$(find pr2_description)/urdf/head_v0/head.urdf.xacro" />
@@ -21,5 +21,5 @@
   <include filename="$(find pr2_description)/urdf/torso_v0/torso.urdf.xacro" />
   <!-- PR2 base -->
-  <include filename="$(find pr2_description)/urdf/base_v0/base.urdf.xacro" />
+  <include filename="$(find pr2_billiards_sim)/urdf/ashok/base_v0/base.urdf.xacro" />
   <!-- Head sensors -->
   <include filename="$(find pr2_description)/urdf/sensors/head_sensor_package.urdf.xacro" />
@@ -115,4 +115,5 @@
     <origin xyz=".135 0 .044" rpy="${M_PI/2} ${-32.25*M_PI/180} 0" />
   </xacro:wge100_camera_v0>
+<!--
   <xacro:property name="lever_length" value="0.5"/>
   <xacro:property name="lever_radius" value="0.0075"/>
@@ -122,8 +123,11 @@
   <xacro:property name="lever_izz" value="0.01"/>
   <xacro:property name="lever_offset_z" value="0.03"/>
-  <joint name="lever_ball_joint" type="fixed" >
+  <joint name="lever_ball_joint" type="revolute" >
     <parent link="r_gripper_palm_link" />
     <child link="lever_stick" />
     <origin xyz="0.2 0 0" rpy="0 0 1.56" />
+    <axis xyz="0 0 1"/>
+    <limit lower="-3.14" upper="3.14" effort="10000" velocity="1.0"/>
+    <calibration reference_position="0.0"/>
   </joint>
   <link name="lever_stick">
@@ -148,7 +152,7 @@
   <gazebo reference="lever_stick">
     <material>Gazebo/Wood</material>
-    <turnGravityOff>false</turnGravityOff>
-  </gazebo>
-  <xacro:property name="cue_length" value="1.47"/>
+    <turnGravityOff>true</turnGravityOff>
+  </gazebo>
+  <xacro:property name="cue_length" value="1.0"/>
   <xacro:property name="cue_radius" value="0.0065"/>
   <xacro:property name="cue_mass" value="0.01"/>
@@ -160,7 +164,7 @@
     <parent link="lever_stick" />
     <child link="cue_stick" />
-    <origin xyz="-0.4 0 ${lever_length}" rpy="0 0 0" />
+    <origin xyz="0 0 ${lever_length}" rpy="0 0 0" />
     <axis xyz="0 1 0"/>
-    <limit lower="0.0" upper="1.8" effort="10000" velocity="1.0"/>
+    <limit lower="-3.14" upper="3.14" effort="10000" velocity="1.0"/>
     <calibration reference_position="0.0"/>
   </joint>
@@ -186,5 +190,5 @@
   <gazebo reference="cue_stick">
     <material>Gazebo/Wood</material>
-    <turnGravityOff>false</turnGravityOff>
+    <turnGravityOff>true</turnGravityOff>
   </gazebo>
   <xacro:property name="bridge_mass" value="0.1"/>
@@ -221,5 +225,5 @@
   <gazebo reference="bridge">
     <material>Gazebo/White</material>
-    <turnGravityOff>false</turnGravityOff>
+    <turnGravityOff>true</turnGravityOff>
     <selfCollide>true</selfCollide>
   </gazebo>
@@ -250,5 +254,5 @@
   <gazebo reference="bridge_bottom">
     <material>Gazebo/Red</material>
-    <turnGravityOff>false</turnGravityOff>
+    <turnGravityOff>true</turnGravityOff>
     <selfCollide>true</selfCollide>
   </gazebo>
@@ -263,3 +267,9 @@
 <mechanicalReduction>1.0</mechanicalReduction>
 </transmission>
+<transmission name="lever_ball_bridge" type="SimpleTransmission">
+<actuator name="lb"/>
+<joint name="lever_ball_joint"/>
+<mechanicalReduction>1.0</mechanicalReduction>
+</transmission>
+-->
 </robot>

Commit message: Made grasping of stick and bridge possible

File: pr2_billiards_sim/urdf/pr2.urdf.xacro (robot description, xacro)
@@ -277,9 +277,9 @@
 <mechanicalReduction>1.0</mechanicalReduction>
 </transmission>
-<!--transmission name="cue_bridge" type="SimpleTransmission">
+<transmission name="cue_bridge" type="SimpleTransmission">
 <actuator name="cb"/>
 <joint name="cue_bridge_joint"/>
 <mechanicalReduction>1.0</mechanicalReduction>
-</transmission-->
+</transmission>
 <transmission name="lever_ball_bridge" type="SimpleTransmission">
 <actuator name="lb"/>

File: pr2_billiards_sim/urdf/stick.urdf.xacro (robot description, xacro)
@@ -79,8 +79,72 @@
   <joint name="cue_bridge_joint" type="prismatic" >
     <parent link="cue_stick" />
+    <child link="link_virtual1" />
+    <origin xyz="0 0 ${cue_length-0.05}" rpy="0 0 0" />
+    <axis xyz="0 0 1"/>
+    <limit lower="-0.1" upper="0.1" effort="10000" velocity="1.0"/>
+    <calibration reference_position="0.0"/>
+  </joint>
+  <link name="link_virtual1">
+   <inertial>
+      <mass value="${cue_mass/1000}" />
+      <origin xyz="0 0 0" rpy="0 0 0" />
+      <inertia  ixx="0" ixy="0.0"  ixz="0.01"  iyy="0.01"  iyz="0.0"  izz="0.01" />
+    </inertial>
+    <visual>
+      <origin xyz="0.0 0 0" rpy="0 0 0" />
+      <geometry>
+        <cylinder length="0.01" radius="0.01"/>
+      </geometry>
+    </visual>
+    <collision>
+      <origin xyz="0.01 0 0" rpy="0 0 0" />
+      <geometry>
+        <cylinder length="0.01" radius="0.01"/>
+      </geometry>
+    </collision>
+  </link>
+  <gazebo reference="link_virtual1">
+    <material>Gazebo/Wood</material>
+    <turnGravityOff>true</turnGravityOff>
+  </gazebo>
+  <!-- This joint allows pitching of the bridge-->
+  <joint name="virtual_rev_joint_1" type="revolute" >
+    <parent link="link_virtual1" />
+    <child link="link_virtual2" />
+    <origin xyz="0 0 0" rpy="0 0 0" />
+    <axis xyz="0 1 0"/>
+    <limit lower="-0.5" upper="0.5" effort="10000" velocity="2.0"/>
+    <calibration reference_position="0.0"/>
+  </joint>
+  <link name="link_virtual2">
+<inertial>
+      <mass value="${cue_mass/1000}" />
+      <origin xyz="0 0 0" rpy="0 0 0" />
+      <inertia  ixx="0" ixy="0.0"  ixz="0.01"  iyy="0.01"  iyz="0.0"  izz="0.01" />
+    </inertial>
+    <visual>
+      <origin xyz="0.0 0 0" rpy="0 0 0" />
+      <geometry>
+        <cylinder length="0.01" radius="0.01"/>
+      </geometry>
+    </visual>
+    <collision>
+      <origin xyz="0.01 0 0" rpy="0 0 0" />
+      <geometry>
+        <cylinder length="0.01" radius="0.01"/>
+      </geometry>
+    </collision>
+  </link>
+  <gazebo reference="link_virtual2">
+    <material>Gazebo/Wood</material>
+    <turnGravityOff>true</turnGravityOff>
+  </gazebo>
+  <!-- This joint allows yawing of the bridge-->
+  <joint name="virtual_rev_joint_2" type="revolute" >
+    <parent link="link_virtual2" />
     <child link="bridge" />
-    <origin xyz="0 0 ${cue_length-0.05}" rpy="1.57 0 0" />
-    <axis xyz="0 1 0"/>
-    <limit lower="-0.1" upper="0.1" effort="10000" velocity="1.0"/>
+    <origin xyz="0 0 0" rpy="0 0 0" />
+    <axis xyz="1 0 0"/>
+    <limit lower="-0.5" upper="0.5" effort="10000" velocity="2.0"/>
     <calibration reference_position="0.0"/>
   </joint>
@@ -100,5 +164,5 @@
       <origin xyz="-0.06 0 0" rpy="0 0 0" />
       <geometry>
-        <box size="0.10 0.03 0.005"/>
+        <box size="0.10 0.04 0.005"/>
       </geometry>
     </collision>
@@ -143,8 +207,18 @@
 <mechanicalReduction>1.0</mechanicalReduction>
 </transmission>
-<transmission name="cue_bridge" type="SimpleTransmission">
+<transmission name="cue_v1" type="SimpleTransmission">
 <actuator name="cb"/>
 <joint name="cue_bridge_joint"/>
 <mechanicalReduction>1.0</mechanicalReduction>
 </transmission>
+<transmission name="v1_v2" type="SimpleTransmission">
+<actuator name="v12"/>
+<joint name="virtual_rev_joint_1"/>
+<mechanicalReduction>1.0</mechanicalReduction>
+</transmission>
+<transmission name="v2_bridge" type="SimpleTransmission">
+<actuator name="v2b"/>
+<joint name="virtual_rev_joint_2"/>
+<mechanicalReduction>1.0</mechanicalReduction>
+</transmission>
 </robot>
