Commit message: Add cue stick as known object to ROS

File: pr2_billiards_sim/urdf/stick.urdf.xacro (robot description, xacro)
@@ -158,5 +158,5 @@
       <origin xyz="-0.06 0 0" rpy="0 0 0" />
       <geometry>
-        <box size="0.10 0.04 0.005"/>
+        <box size="0.10 0.07 0.005"/>
       </geometry>
     </visual>
@@ -164,5 +164,5 @@
       <origin xyz="-0.06 0 0" rpy="0 0 0" />
       <geometry>
-        <box size="0.10 0.04 0.005"/>
+        <box size="0.10 0.07 0.005"/>
       </geometry>
     </collision>
